File: power_prong.sch (EAGLE design)
At the start: 19 parts, among them IC1 INA138, IC2 MCP1824S, Q1 FDG332PZ, X1 USBSMD

Commit message: Resize for panelizing
Parts:
- removed LOGO1: LOGO_CC-BY-SA, dp_devices:LOGO_CC-BY-SA
Changed lines of the file:
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@@
 <part name="TP1" library="SparkFun-Connectors" deviceset="M02" device="3.5MM-NO_SILK"/>
 <part name="FRAME1" library="space_age_robotics" deviceset="FRAME-LETTER" device=""/>
-<part name="LOGO1" library="dp_devices" deviceset="LOGO_CC-BY-SA" device=""/>
 </parts>
 <sheets>
@@
 <instance part="FRAME1" gate="G$1" x="-63.5" y="-60.96"/>
 <instance part="FRAME1" gate="G$2" x="83.82" y="-60.96"/>
-<instance part="LOGO1" gate="LOGO" x="71.12" y="-55.88"/>
 </instances>
 <busses>
